Commit message: gabut

File: src/conveyorbelt_models/models/conveyor_belt_model.urdf (robot description, URDF)
Before this commit: robot conveyor_belt_model, 4 links, 3 joints
Links:
- link another_link: mass 0.3 -> 0.05
- link base_link: mass 1.2 -> 1.0
- link belt_link: mass 0.5 -> 0.2
- link motor_link: mass 0.3 -> 0.05

File: src/conveyorbelt_models/models/conveyor_belt_model2.urdf (robot description, URDF)
Before this commit: robot conveyor_belt_model2, 4 links, 3 joints
Links:
- link base_link_convey2: mass 1.3 -> 1.8
- link convey2_another_link: mass 0.3 -> 0.05
- link convey2_belt_link: mass 0.5 -> 0.2
- link convey2_motor_link: mass 0.3 -> 0.05
