Commit message: ujicoba 1

File: src/conveyorbelt_models/models/box_model.urdf (robot description, URDF)
Before this commit: robot box_model, 1 links, 0 joints
Links:
- link box_link: mass 0.124 -> 0.013

File: src/conveyorbelt_models/models/conveyor_belt_model.urdf (robot description, URDF)
Before this commit: robot conveyor_belt_model, 4 links, 3 joints
Links:
- link base_link: mass 1.0 -> 0.102
- link belt_link: mass 0.2 -> 0.024
Joints:
- joint another_joint: limit effort=100 velocity=2.2 -> effort=100 velocity=1.625
- joint belt_joint: limit effort=100 velocity=2.2 -> effort=100 velocity=1.625
- joint motor_joint: limit effort=100 velocity=2.2 -> effort=100 velocity=1.625

File: src/conveyorbelt_models/models/conveyor_belt_model2.urdf (robot description, URDF)
Before this commit: robot conveyor_belt_model2, 4 links, 3 joints
Links:
- link base_link_convey2: mass 1.8 -> 0.184
- link convey2_belt_link: mass 0.2 -> 0.024
Joints:
- joint convey2_another_joint: limit effort=100 velocity=2.2 -> effort=100 velocity=1.925
- joint convey2_belt_joint: limit lower=0 upper=0 effort=100 velocity=2.2 -> lower=0 upper=0 effort=100 velocity=1.925
- joint convey2_motor_joint: limit effort=100 velocity=2.2 -> effort=100 velocity=1.925

Commit message: 2022

File: src/conveyorbelt_models/models/box_model.urdf (robot description, URDF)
Before this commit: robot box_model, 1 links, 0 joints
Links:
- link box_link: mass 0.013 -> 0.014

File: src/conveyorbelt_models/models/box_model_store.urdf (robot description, URDF)
Before this commit: robot box_store_model, 1 links, 0 joints
Links:
- link box_link: mass 0.124 -> 0.013

File: src/conveyorbelt_models/models/conveyor_belt_model.urdf (robot description, URDF)
Before this commit: robot conveyor_belt_model, 4 links, 3 joints
Joints:
- joint another_joint: limit effort=100 velocity=1.625 -> effort=100 velocity=1.8
- joint belt_joint: limit effort=100 velocity=1.625 -> effort=100 velocity=1.8
- joint motor_joint: limit effort=100 velocity=1.625 -> effort=100 velocity=1.8
